Commit message: AEB System Done!

File: description/gazebo_control.xacro (robot description, xacro)
@@ -10,6 +10,6 @@
             <wheel_diameter>0.1</wheel_diameter>
             <!-- limits -->
-            <max_wheel_torque>200</max_wheel_torque>
-            <max_wheel_acceleration>10.0</max_wheel_acceleration>
+            <max_wheel_torque>10</max_wheel_torque>
+            <max_wheel_acceleration>1.0</max_wheel_acceleration>
             <!-- outputs -->
             <odometry_frame>odom</odometry_frame>

File: description/lidar.xacro (robot description, xacro)
@@ -37,5 +37,5 @@
 												<!--resolution>: this number is multiplied by samples to determine the number range data points.-->
                         <resolution>1</resolution>
-							          <min_angle>-3.14</min_angle>
+						<min_angle>-3.14</min_angle>
                         <max_angle>3.14</max_angle>
                     </horizontal>
@@ -43,5 +43,5 @@
                 <range>
                     <min>0.3</min>
-                    <max>2</max>
+                    <max>12</max>
                     <resolution>0.01</resolution>
                 </range>

File: description/robot_core.xacro (robot description, xacro)
@@ -83,8 +83,8 @@
             <origin xyz="0 0 0" rpy="0 0 0"/>
         </xacro:inertial_cylinder>
-        <gazebo reference="right_wheel">
+    </link>
+    <gazebo reference="right_wheel">
             <material>Gazebo/Blue</material>
-        </gazebo>
-    </link>
+    </gazebo>
     <!-- caster wheel joint -->
     <joint name="caster_wheel_joint" type="fixed">
@@ -109,9 +109,9 @@
             <origin xyz="0 0 0" rpy="0 0 0"/>
         </xacro:inertial_sphere>
-        <gazebo reference="caster_wheel">
+    </link>
+    <gazebo reference="caster_wheel">
             <material>Gazebo/Black</material>
             <mu1 value = "0.001" />
             <mu2 value = "0.001" />
-        </gazebo>
-    </link>
+    </gazebo>
 </robot>
