Commit message: se implementó el ros2control pero me aparece un error al leer la configuración my_controllers.yaml

File: description/properties.xacro (robot description, xacro)
@@ -14,3 +14,6 @@
         <color rgba= "0 0 0 1"/>
     </material>
+    <material name="red">
+        <color rgba="1.0 0.0 0.0 1.0"/>
+    </material>
 </robot>

File: description/robot.urdf.xacro (robot description, xacro)
@@ -3,4 +3,5 @@
     <!-- Example link -->
     <xacro:include filename="robot_core.xacro"/>
+    <xacro:include filename="ros2_control.xacro"/>
     <xacro:include filename="properties.xacro"/>
     <xacro:include filename="inertial_macros.xacro"/>

File: description/robot_core.xacro (robot description, xacro)
@@ -6,5 +6,5 @@
     <link name="base_link">
     </link>
-    <joint name="base_link" type="fixed">
+    <joint name="base_link_joint" type="fixed">
         <parent link="base_link"/>
         <child link="chassis"/>
