Commit message: Distance finder done!

File: description/lidar.xacro (robot description, xacro)
@@ -37,11 +37,11 @@
 												<!--resolution>: this number is multiplied by samples to determine the number range data points.-->
                         <resolution>1</resolution>
-						<min_angle>-3.14</min_angle>
-                        <max_angle>3.14</max_angle>
+						<min_angle>-1.57</min_angle>
+                        <max_angle>1.57</max_angle>
                     </horizontal>
                 </scan>
                 <range>
                     <min>0.3</min>
-                    <max>12</max>
+                    <max>3</max>
                     <resolution>0.01</resolution>
                 </range>

File: description/robot_core.xacro (robot description, xacro)
@@ -29,8 +29,8 @@
             <origin xyz="0.15 0 0.075" rpy="0 0 0"/>
         </xacro:inertial_box>
-        <gazebo reference="chassis">
+    </link>
+    <gazebo reference="chassis">
             <material>Gazebo/White</material>
         </gazebo>
-    </link>
     <!-- left wheel joint -->
     <joint name="left_wheel_joint" type="continuous">
@@ -56,8 +56,8 @@
             <origin xyz="0 0 0" rpy="0 0 0"/>
         </xacro:inertial_cylinder>
-        <gazebo reference="left_wheel">
+    </link>
+    <gazebo reference="left_wheel">
             <material>Gazebo/Blue</material>
         </gazebo>
-    </link>
     <!-- right wheel joint -->
     <joint name="right_wheel_joint" type="continuous">

Commit message: Ya se tiene funcionando para el path tracking el waypoints tracking

File: description/lidar.xacro (robot description, xacro)
@@ -37,11 +37,11 @@
 												<!--resolution>: this number is multiplied by samples to determine the number range data points.-->
                         <resolution>1</resolution>
-						<min_angle>-1.57</min_angle>
-                        <max_angle>1.57</max_angle>
+                        <min_angle>-3.14159</min_angle>
+                        <max_angle>3.14159</max_angle>
                     </horizontal>
                 </scan>
                 <range>
-                    <min>0.1</min>
-                    <max>2.5</max>
+                    <min>0.3</min>
+                    <max>20.0</max>
                     <resolution>0.01</resolution>
                 </range>

File: description/properties.xacro (robot description, xacro)
@@ -14,3 +14,6 @@
         <color rgba= "0 0 0 1"/>
     </material>
+    <material name="red">
+        <color rgba= "1 0 0 1"/>
+    </material>
 </robot>

File: description/robot_core.xacro (robot description, xacro)
@@ -6,4 +6,12 @@
     <link name="base_link">
     </link>
+    <!-- base_footprint link -->
+    <link name="base_footprint">
+    </link>
+    <joint name="base_footprint_joint" type="fixed">
+        <parent link="base_link"/>
+        <child link="base_footprint"/>
+        <origin xyz="0 0 0" rpy="0 0 0"/>
+    </joint>
     <joint name="base_link" type="fixed">
         <parent link="base_link"/>
